Commit message: Defined a new link so tool frame is at end effector tip

File: src/panda_arm_moveit/urdf/panda.urdf (robot description, URDF)
Before this commit: robot panda, 12 links, 11 joints
Links:
- added link tool0
Joints:
- added joint tool0_joint: type fixed, parent panda_hand, child tool0, origin xyz=0 0 0.1034 rpy=0 0 0
