Commit message: Add the Universal Robots UR3e (robot:=ur3e); UR arms use UR's visual meshes
ur3e.urdf from UR's UR3e kinematics, limits (wrist 3 continuous) and meshes; its home keeps the Panda home's camera
orientation and x/y at z = 0.30 m, since the 500 mm reach can't get to the Panda's 0.51 m. Both UR arms now show UR's
.dae visual meshes; collision checks still use the collision meshes.

Co-Authored-By: Claude Opus 5.5 <noreply@anthropic.com>

File: src/ur_arm_moveit/urdf/ur5e.urdf (robot description, URDF)
Before this commit: robot ur5e, 10 links, 9 joints
Links:
- link base_link_inertia: geometry collision mesh filename=package://ur_arm_moveit/meshes/ur5e/base.stl; visual mesh filename=package://ur_arm_moveit/meshes/ur5e/visual/base.dae
- link forearm_link: geometry collision mesh filename=package://ur_arm_moveit/meshes/ur5e/forearm.stl; visual mesh filename=package://ur_arm_moveit/meshes/ur5e/visual/forearm.dae
- link shoulder_link: geometry collision mesh filename=package://ur_arm_moveit/meshes/ur5e/shoulder.stl; visual mesh filename=package://ur_arm_moveit/meshes/ur5e/visual/shoulder.dae
- link upper_arm_link: geometry collision mesh filename=package://ur_arm_moveit/meshes/ur5e/upperarm.stl; visual mesh filename=package://ur_arm_moveit/meshes/ur5e/visual/upperarm.dae
- link wrist_1_link: geometry collision mesh filename=package://ur_arm_moveit/meshes/ur5e/wrist1.stl; visual mesh filename=package://ur_arm_moveit/meshes/ur5e/visual/wrist1.dae
- link wrist_2_link: geometry collision mesh filename=package://ur_arm_moveit/meshes/ur5e/wrist2.stl; visual mesh filename=package://ur_arm_moveit/meshes/ur5e/visual/wrist2.dae
- link wrist_3_link: geometry collision mesh filename=package://ur_arm_moveit/meshes/ur5e/wrist3.stl; visual mesh filename=package://ur_arm_moveit/meshes/ur5e/visual/wrist3.dae
