Commit message: ur3e: 5 cm long, 1 cm wide camera tube (tool0 0.0534 m from the flange); home recomputed for the same camera pose
Co-Authored-By: Claude Opus 5.5 <noreply@anthropic.com>

File: src/ur_arm_moveit/urdf/ur3e.urdf (robot description, URDF)
Before this commit: robot ur3e, 10 links, 9 joints
Links:
- link camera: geometry collision cylinder length=0.05 radius=0.005; visual cylinder length=0.05 radius=0.005
Joints:
- joint tool0_joint: origin xyz=0 0 0.1034 rpy=0 0 0 -> xyz=0 0 0.0534 rpy=0 0 0
